File: PCB_design/Low-level-driver/Low-level-driver.kicad_sch (KiCad schematic)
At the start: 59 parts, among them J101 Conn_01x02, J102 Conn_01x05, J103 Conn_01x04, Q101 NMOS, Q102 NMOS, Q103 NMOS, Q104 NMOS, U101 AD5280BRUZ20, U102 AD5280BRUZ20, U103 LM5143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

Commit message: Schematic hierarchical redesign
Parts:
- removed C101, C106, C107, C108, C109, C114, C115, C116: C, symbol Device:C
- removed C102, C103, C104, C105, C113, C117, C119: 10u, symbol Device:C
- removed C110, C112: 0.1uF, symbol Device:C
- removed C111: 470n, symbol Device:C
- removed C118: 10n, symbol Device:C
- removed C120: 1u, symbol Device:C
- removed C121, C122, C123: 4.7u, symbol Device:C
- removed D101, D102: D_Schottky, symbol Device:D_Schottky
- removed J103: Conn_01x04, symbol Connector_Generic:Conn_01x04
- removed L101, L102: L, symbol Device:L
- removed Q101, Q102, Q103, Q104: NMOS, symbol Simulation_SPICE:NMOS
- removed R102, R103, R107, R109, R112: 10k, symbol Device:R
- removed R104, R105: 18k, symbol Device:R
- removed R106, R108, R110, R111, R113, R118, R119: R, symbol Device:R
- removed R114: 100k, symbol Device:R
- removed R115: 11k, symbol Device:R
- removed U101, U102: AD5280BRUZ20, Package_SO:TSSOP-14_4.4x5mm_P0.65mm, symbol Potentiometer_Digital:AD5280
- removed U103: LM5143, Lab_source:Texas_RHA0040P_VQFN-40-1EP_6x6mm_P0.5mm_EP4.15x4.15mm_ThermalVias, symbol Power_source:LM5143
- removed U104: TCA9535PWR, Package_SO:TSSOP-24_4.4x7.8mm_P0.65mm, symbol Interface_Expansion:TCA9535PWR
- removed U105: TPS7A4101DGN, Package_SO:Texas_DGN0008B_VSSOP-8-1EP_3x3mm_P0.65mm_EP2x3mm_Mask1.88x1.98mm_ThermalVias, symbol Regulator_Linear:TPS7A4101DGN
- removed U106: LM27761, Package_SON:WSON-8-1EP_2x2mm_P0.5mm_EP0.9x1.6mm, symbol Regulator_SwitchedCapacitor:LM27761
- added J102, J103: Conn_01x02, symbol Connector_Generic:Conn_01x02
- J104: renamed from J102; value Conn_01x05 -> Conn_01x06; symbol Connector_Generic:Conn_01x05 -> Connector_Generic:Conn_01x06
- renumbered R116 to R102, R117 to R103
Connections:
- net GND: now also J104.3 (Pin_3), J102.2 (Pin_2), J103.2 (Pin_2); no longer J104.2 (Pin_2)
- net SCL: now also J104.4 (Pin_4); no longer J104.3 (Pin_3)
- net SDA: now also J104.5 (Pin_5); no longer J104.4 (Pin_4)
- net ~{INT_{TCA}}: now also J104.6 (Pin_6); no longer J104.5 (Pin_5)
- net V_{out1}.FB: no longer names the net of R101.1
- new net +5V: J104.2 (Pin_2)
- new net Output Enable 1/V_{out}: J102.1 (Pin_1)
- new net Output Enable 2/V_{out}: J103.1 (Pin_1)
- no-connect marks 5 -> 2
Other:
- removed sheet Ballast
- removed sheet Ballast1
- removed sheet Output Enable - V_{OUT1}
- removed sheet Output Enable - V_{OUT2}
- added sheet Auxiliary power supply (auxiliary_power_supply.kicad_sch)
- added sheet Feedback loop 1 (feedback_loop.kicad_sch)
- added sheet Feedback loop 2 (feedback_loop.kicad_sch)
- added sheet Filter_{OUT} 1 (emi_output.kicad_sch)
- added sheet Filter_{OUT} 2 (emi_output.kicad_sch)
- added sheet Filter_{in} (emi_input.kicad_sch)
- added sheet GPIO expander (gpio_expander.kicad_sch)
- added sheet Output Enable 1 (output_enable.kicad_sch)
- added sheet Output Enable 2 (output_enable.kicad_sch)
- added sheet Power Meter 1 (power_meter.kicad_sch)
- added sheet Power Meter 2 (power_meter.kicad_sch)
- added sheet Power Meter 3 (power_meter.kicad_sch)
- added sheet Power supply (power_supply.kicad_sch)
- note added: "I^{2}C address 0x20"
- note added: "I^{2}C address 0x40"
- note added: "I^{2}C address 0x41"
- note added: "I^{2}C address 0x45"
- note removed: "Feedback loop 1"
- note removed: "Feedback loop 2"
- note removed: "GPIO expander"
- note removed: "Output enable - V_{OUT1}"
- note removed: "Output enable - V_{OUT2}"
- note removed: "Ultra low I_{Q} **NOT** required -> MODE - AGND"
- moved on the sheet: J101, R102, R103
