File: PCB_design/Low-level-driver/ballast2.kicad_sch (KiCad schematic)
At the start: 36 parts, among them Q701 BC846BPN, Q702 BC846BPN, Q703 BC846BPN, Q704 BC846BPN, Q705 BC846BPN, Q706 BC846BPN, Q707 BC846BPN, Q708 BC846BPN, U701 TMUX1208PWR

Commit message: Schematic hierarchical redesign
Parts:
- renumbered Q701 to Q1301, Q702 to Q1302, Q703 to Q1303, Q704 to Q1304, Q705 to Q1305, Q706 to Q1306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
Connections:
- net Ballast.in renamed V_{IN}
- net Ballast.out renamed V_{OUT}
Other:
- title: (none) -> Power supply - low level driver
