File: PCB_design/Low-level-driver/to_be_removed.kicad_sch (KiCad schematic)
At the start: 47 parts, among them J501 Conn_01x02, J502 Conn_01x02, Q501 Q_NMOS_DGS, Q502 Q_NMOS_DGS, Q503 Q_NMOS_DGS, Q504 Q_NMOS_DGS, U501 LM5175PWP, U502 AD5280BRUZ20

Commit message: Schematic hierarchical redesign
Parts:
- renumbered C501 to C1901, C502 to C1902, C503 to C1903, C504 to C1904, C505 to C1905, C506 to C1906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
Other:
- title: (none) -> Power supply - low level driver
