File: PCB_design/Low-level-driver/emi_input.kicad_sch (KiCad schematic)
At the start: 1 part

Commit message: Initial thesis release
Connections:
- net IN: no longer C1001.1
- new net OUT: C1001.1
Changed lines of the file:
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@@
 (kicad_sch
-	(version 20231120)
+	(version 20250114)
 	(generator "eeschema")
-	(generator_version "8.0")
+	(generator_version "9.0")
 	(paper "A4")
 	(title_block
@@
 		(date "2024-06-28")
 	)
-	(junction
-		(at 153.67 87.63)
-		(diameter 0)
-		(color 0 0 0 0)
-	)
 	(wire
 		(pts
 			(xy 153.67 87.63) (xy 176.53 87.63)
-		)
-		(stroke
-			(width 0)
-			(type default)
-		)
-	)
-	(wire
-		(pts
-			(xy 50.8 87.63) (xy 153.67 87.63)
 		)
 		(stroke
@@
 		)
 	)
+	(wire
+		(pts
+			(xy 50.8 87.63) (xy 60.96 87.63)
+		)
+		(stroke
+			(width 0)
+			(type default)
+		)
+	)
 	(hierarchical_label "IN"
 		(shape input)
 		(at 50.8 87.63 180)
-		(fields_autoplaced yes)
 		(effects
 			(font
@@
 		(shape output)
 		(at 176.53 87.63 0)
-		(fields_autoplaced yes)
 		(effects
 			(font
