File: PCB_design/Power_unit/Power_unit_A1/ballast.kicad_sch (KiCad schematic)
At the start: 36 parts, among them Q1301 BC846BPN, Q1302 BC846BPN, Q1303 BC846BPN, Q1304 BC846BPN, Q1305 BC846BPN, Q1306 BC846BPN, Q1307 BC846BPN, Q1308 BC846BPN, U1301 TMUX1208PWR

Commit message: Initial thesis release
Parts:
- removed Q1301, Q1302, Q1303, Q1304, Q1305, Q1306, Q1307, Q1308: BC846BPN, Package_TO_SOT_SMD:SOT-363_SC-70-6, symbol Transistor_BJT:BC846BPN
- removed R1301, R1303, R1304, R1306, R1307, R1309, R1310, R1313, R1314, R1317, R1318, R1320, R1321, R1324, R1325: 100k, symbol Device:R
- removed R1302: 2k2, symbol Device:R
- removed R1305, R1311, R1323: 200k, symbol Device:R
- removed R1308, R1312, R1315, R1316, R1327: 400k, symbol Device:R
- removed R1319, R1322, R1326: 1M, symbol Device:R
- removed U1301: TMUX1208PWR, Package_SO:TSSOP-16_4.4x5mm_P0.65mm, symbol Lab_supply:TMUX1208PWR
- added Q401, Q402, Q403, Q404, Q405, Q406, Q407, Q408: BC846BPN, Package_TO_SOT_SMD:SOT-363_SC-70-6, symbol Transistor_BJT:BC846BPN
- added R401, R403, R406, R409, R413, R417, R420, R424: 10k, symbol Device:R
- added R402: 2k2, symbol Device:R
- added R404, R407, R410, R414, R418, R421, R425: 100k, symbol Device:R
- added R405, R411, R423: 200k, symbol Device:R
- added R408, R412, R415, R416, R427: 400k, symbol Device:R
- added R419, R422, R426: 1M, symbol Device:R
- added U401: TMUX1208PWR, Package_SO:TSSOP-16_4.4x5mm_P0.65mm, symbol Lab_supply:TMUX1208PWR
Connections:
- net +3V3: now also U401.13 (VDD), U401.2 (EN), U401.8 (D)
- net A0: now also U401.1 (A0)
- net A1: now also U401.16 (A1)
- net A2: now also U401.15 (A2)
- net GND: now also Q401.1 (E1), Q402.1 (E1), Q403.1 (E1), Q404.1 (E1), Q405.1 (E1), Q406.1 (E1), Q407.1 (E1), Q408.1 (E1), U401.14 (GND)
- net V_{IN}: now also Q401.4 (E2), Q402.4 (E2), Q403.4 (E2), Q404.4 (E2), Q405.4 (E2), Q406.4 (E2), Q407.4 (E2), Q408.4 (E2)
- net V_{OUT}: now also Q401.3 (C2), R405.2, R408.2, R412.2, R416.2, R419.2, R423.2, R427.2
- net ball.stg.0: now also R401.2, U401.4 (S1)
- net ball.stg.1: now also R403.2, U401.5 (S2)
- net ball.stg.2: now also R406.2, U401.6 (S3)
- net ball.stg.3: now also R409.2, U401.7 (S4)
- net ball.stg.4: now also R413.2, U401.12 (S5)
- net ball.stg.5: now also R417.2, U401.11 (S6)
- net ball.stg.6: now also R420.2, U401.10 (S7)
- net ball.stg.7: now also R424.2, U401.9 (S8)
- new net: Q403.2 (B1), R406.1
- new net: Q403.6 (C1), R407.2
- new net: Q407.3 (C2), R422.1
- new net: Q407.5 (B2), R421.1
- new net: Q401.5 (B2), R402.1
- new net: Q404.3 (C2), R411.1
- new net: R411.2, R412.1
- new net: Q408.2 (B1), R424.1
- new net: Q405.3 (C2), R415.1
- new net: R415.2, R416.1
- new net: Q404.5 (B2), R410.1
- new net: Q404.6 (C1), R410.2
- new net: Q405.5 (B2), R414.1
- new net: Q406.3 (C2), R419.1
- new net: Q406.5 (B2), R418.1
- new net: Q403.3 (C2), R408.1
- new net: Q403.5 (B2), R407.1
- new net: Q402.3 (C2), R405.1
- new net: Q402.5 (B2), R404.1
- new net: Q405.6 (C1), R414.2
- new net: Q405.2 (B1), R413.1
- new net: Q401.2 (B1), R401.1
- new net: R422.2, R423.1
- new net: Q402.6 (C1), R404.2
- new net: Q408.5 (B2), R425.1
- new net: Q408.6 (C1), R425.2
- new net: Q407.6 (C1), R421.2
- new net: R426.2, R427.1
- new net: Q402.2 (B1), R403.1
- new net: Q406.2 (B1), R417.1
- new net: Q408.3 (C2), R426.1
- new net: Q407.2 (B1), R420.1
- new net: Q406.6 (C1), R418.2
- new net: Q401.6 (C1), R402.2
- new net: Q404.2 (B1), R409.1
