File: PCB_design/Power_unit/Power_unit_A1/feedback_loop.kicad_sch (KiCad schematic)
At the start: 5 parts, among them U301 AD5280BRUZ20

Commit message: Initial thesis release
Other:
- sheet Ballast: file ballast2.kicad_sch -> ballast.kicad_sch
- moved on the sheet: C301, C302, R301, R302, U301
