File: PCB_design/Power_unit/Power_unit_A1/output_enable.kicad_sch (KiCad schematic)
At the start: 6 parts, among them Q501 Q_NPN_EBC, Q502 PMOS

Commit message: Initial thesis release
Parts:
- renumbered D501 to D1501, Q501 to Q1501, Q502 to Q1502, R501 to R1501, R502 to R1502, R503 to R1503
Changed lines of the file:
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@@
 		(dnp no)
 		(fields_autoplaced yes)
-		(property "Reference" "R503"
+		(property "Reference" "R1503"
 			(at 85.09 83.8199 0)
 			(effects
@@
 		)
 		(instances
-			(project "Low-level-driver"
-				(path "/2e43a8c9-1b23-4896-a481-133b23afb346/016df87f-c803-44fb-9ff3-a33dc71d7c4c"
-					(reference "R603")
-					(unit 1)
-				)
-				(path "/2e43a8c9-1b23-4896-a481-133b23afb346/9363c3cd-da89-4013-abbb-a8f39df5ef51"
-					(reference "R503")
+			(project "Power_unit_A1"
+				(path "/39e95423-af83-4645-98fc-4a660ba074aa/601d2e12-3ced-43d7-94eb-d0cf5634b17c"
+					(reference "R1503")
+					(unit 1)
+				)
+				(path "/39e95423-af83-4645-98fc-4a660ba074aa/cb7ffc2b-1dcf-4375-80b8-18d54c0176ff"
+					(reference "R1603")
 					(unit 1)
 				)
@@
 		(on_board yes)
 		(dnp no)
-		(property "Reference" "Q502"
+		(property "Reference" "Q1502"
 			(at 82.55 59.69 90)
 			(effects
@@
 		)
 		(instances
-			(project "Low-level-driver"
-				(path "/2e43a8c9-1b23-4896-a481-133b23afb346/016df87f-c803-44fb-9ff3-a33dc71d7c4c"
-					(reference "Q602")
-					(unit 1)
-				)
-				(path "/2e43a8c9-1b23-4896-a481-133b23afb346/9363c3cd-da89-4013-abbb-a8f39df5ef51"
-					(reference "Q502")
+			(project "Power_unit_A1"
+				(path "/39e95423-af83-4645-98fc-4a660ba074aa/601d2e12-3ced-43d7-94eb-d0cf5634b17c"
+					(reference "Q1502")
+					(unit 1)
+				)
+				(path "/39e95423-af83-4645-98fc-4a660ba074aa/cb7ffc2b-1dcf-4375-80b8-18d54c0176ff"
+					(reference "Q1602")
 					(unit 1)
 				)
@@
 		(dnp no)
 		(fields_autoplaced yes)
-		(property "Reference" "R501"
+		(property "Reference" "R1501"
 			(at 59.69 69.8499 0)
 			(effects
@@
 		)
 		(instances
-			(project "Low-level-driver"
-				(path "/2e43a8c9-1b23-4896-a481-133b23afb346/016df87f-c803-44fb-9ff3-a33dc71d7c4c"
-					(reference "R601")
-					(unit 1)
-				)
-				(path "/2e43a8c9-1b23-4896-a481-133b23afb346/9363c3cd-da89-4013-abbb-a8f39df5ef51"
-					(reference "R501")
+			(project "Power_unit_A1"
+				(path "/39e95423-af83-4645-98fc-4a660ba074aa/601d2e12-3ced-43d7-94eb-d0cf5634b17c"
+					(reference "R1501")
+					(unit 1)
+				)
+				(path "/39e95423-af83-4645-98fc-4a660ba074aa/cb7ffc2b-1dcf-4375-80b8-18d54c0176ff"
+					(reference "R1601")
 					(unit 1)
 				)
@@
 		(on_board yes)
 		(dnp no)
-		(property "Reference" "R502"
+		(property "Reference" "R1502"
 			(at 69.85 92.964 90)
 			(effects
@@
 		)
 		(instances
-			(project "Low-level-driver"
-				(path "/2e43a8c9-1b23-4896-a481-133b23afb346/016df87f-c803-44fb-9ff3-a33dc71d7c4c"
-					(reference "R602")
-					(unit 1)
-				)
-				(path "/2e43a8c9-1b23-4896-a481-133b23afb346/9363c3cd-da89-4013-abbb-a8f39df5ef51"
-					(reference "R502")
+			(project "Power_unit_A1"
+				(path "/39e95423-af83-4645-98fc-4a660ba074aa/601d2e12-3ced-43d7-94eb-d0cf5634b17c"
+					(reference "R1502")
+					(unit 1)
+				)
+				(path "/39e95423-af83-4645-98fc-4a660ba074aa/cb7ffc2b-1dcf-4375-80b8-18d54c0176ff"
+					(reference "R1602")
 					(unit 1)
 				)
@@
 		(dnp no)
 		(fields_autoplaced yes)
-		(property "Reference" "Q501"
+		(property "Reference" "Q1501"
 			(at 85.09 93.9799 0)
 			(effects
@@
 		)
 		(instances
-			(project "Low-level-driver"
-				(path "/2e43a8c9-1b23-4896-a481-133b23afb346/016df87f-c803-44fb-9ff3-a33dc71d7c4c"
-					(reference "Q601")
-					(unit 1)
-				)
-				(path "/2e43a8c9-1b23-4896-a481-133b23afb346/9363c3cd-da89-4013-abbb-a8f39df5ef51"
-					(reference "Q501")
+			(project "Power_unit_A1"
+				(path "/39e95423-af83-4645-98fc-4a660ba074aa/601d2e12-3ced-43d7-94eb-d0cf5634b17c"
+					(reference "Q1501")
+					(unit 1)
+				)
+				(path "/39e95423-af83-4645-98fc-4a660ba074aa/cb7ffc2b-1dcf-4375-80b8-18d54c0176ff"
+					(reference "Q1601")
 					(unit 1)
 				)
@@
 		(dnp no)
 		(fields_autoplaced yes)
-		(property "Reference" "#PWR0501"
+		(property "Reference" "#PWR01501"
 			(at 82.55 97.79 0)
 			(effects
@@
 		)
 		(instances
-			(project "Low-level-driver"
-				(path "/2e43a8c9-1b23-4896-a481-133b23afb346/016df87f-c803-44fb-9ff3-a33dc71d7c4c"
-					(reference "#PWR0601")
-					(unit 1)
-				)
-				(path "/2e43a8c9-1b23-4896-a481-133b23afb346/9363c3cd-da89-4013-abbb-a8f39df5ef51"
-					(reference "#PWR0501")
+			(project "Power_unit_A1"
+				(path "/39e95423-af83-4645-98fc-4a660ba074aa/601d2e12-3ced-43d7-94eb-d0cf5634b17c"
+					(reference "#PWR01501")
+					(unit 1)
+				)
+				(path "/39e95423-af83-4645-98fc-4a660ba074aa/cb7ffc2b-1dcf-4375-80b8-18d54c0176ff"
+					(reference "#PWR01601")
 					(unit 1)
 				)
@@
 		(dnp no)
 		(fields_autoplaced yes)
-		(property "Reference" "D501"
+		(property "Reference" "D1501"
 			(at 69.85 69.8499 90)
 			(effects
@@
 		)
 		(instances
-			(project "Low-level-driver"
-				(path "/2e43a8c9-1b23-4896-a481-133b23afb346/016df87f-c803-44fb-9ff3-a33dc71d7c4c"
-					(reference "D601")
-					(unit 1)
-				)
-				(path "/2e43a8c9-1b23-4896-a481-133b23afb346/9363c3cd-da89-4013-abbb-a8f39df5ef51"
-					(reference "D501")
-					(unit 1)
-				)
+			(project "Power_unit_A1"
+				(path "/39e95423-af83-4645-98fc-4a660ba074aa/601d2e12-3ced-43d7-94eb-d0cf5634b17c"
+					(reference "D1501")
+					(unit 1)
+				)
+				(path "/39e95423-af83-4645-98fc-4a660ba074aa/cb7ffc2b-1dcf-4375-80b8-18d54c0176ff"
+					(reference "D1601")
+					(unit 1)
+				)
