File: PCB_design/Power_unit/Power_unit_A1/Power_unit_A1.kicad_sch (KiCad schematic)
At the start: 10 parts, among them J101 Conn_01x02, J102 Conn_01x02, J103 Conn_01x02, J104 Conn_01x06

Commit message: Initial thesis release
Parts:
- removed NT101, NT102, NT103: NetTie_2, symbol Device:NetTie_2
- removed R101: R, symbol Device:R
- renumbered R102 to R101, R103 to R102
Connections:
- net SCL: now also J104.5 (Pin_5), R102.1; no longer J104.4 (Pin_4), R101.1
- net SDA: now also J104.4 (Pin_4), R101.1; no longer J104.5 (Pin_5), R102.1
- net +48V renamed V_{IN}
- net Output Enable 1/V_{out} renamed Channel Enable - OUT_{1}/V_{out}
- net Output Enable 2/V_{out} renamed Channel Enable - OUT_{2}/V_{out}
- no-connect marks 5 -> 11
Other:
- removed sheet Feedback loop 1
- removed sheet Output Enable 1
- removed sheet Output Enable 2
- added sheet Channel Enable - IN (channel_enable.kicad_sch)
- added sheet Channel Enable - OUT_{1} (channel_enable.kicad_sch)
- added sheet Channel Enable - OUT_{2} (channel_enable.kicad_sch)
- added sheet Feedback loop 3 (feedback_loop2.kicad_sch)
- sheet Feedback loop 2: file feedback_loop.kicad_sch -> feedback_loop2.kicad_sch
- sheet Feedback loop 2 ports: added {I^{2}C}; removed A0, A1, A2
- sheet Filter_{OUT} 1: file emi_output.kicad_sch -> filter_output.kicad_sch
- sheet Filter_{OUT} 2: file emi_output.kicad_sch -> filter_output.kicad_sch
- sheet Filter_{in}: file emi_input.kicad_sch -> filter_input.kicad_sch
- sheet Power supply ports: added none; removed EN_{G}
- note added: "I^{2}C address 0x??"
- note removed: "I^{2}C address 0x2C"
- note removed: "I^{2}C address 0x2F"
- title: Power supply - low level driver -> (none)
- moved on the sheet: J101, J102, J103, J104, R101, R102

Commit message: WIP
Parts:
- added J105, J106, J107: Conn_01x02, symbol Connector_Generic:Conn_01x02
Connections:
- net GND: now also J105.2 (Pin_2), J106.2 (Pin_2), J107.2 (Pin_2)
- net V_{IN}: now also J105.1 (Pin_1)
- net Channel Enable - OUT_{1}/V_{out} renamed V_{OUT1}
- net V_{OUT1}: now also J106.1 (Pin_1)
- net Channel Enable - OUT_{2}/V_{out} renamed V_{OUT2}
- net V_{OUT2}: now also J107.1 (Pin_1)
Other:
- added sheet Auxiliary power supply1 (auxiliary_power_supply.kicad_sch)
- added sheet Channel Enable - IN1 (channel_enable.kicad_sch)
- added sheet Channel Enable - OUT_{1}1 (channel_enable.kicad_sch)
- added sheet Channel Enable - OUT_{2}1 (channel_enable.kicad_sch)
- added sheet Filter_{OUT} 3 (filter_output.kicad_sch)
- added sheet Filter_{OUT} 4 (filter_output.kicad_sch)
- added sheet Filter_{in}1 (filter_input.kicad_sch)
- added sheet Power Meter 4 (power_meter.kicad_sch)
- added sheet Power Meter 5 (power_meter.kicad_sch)
- added sheet Power Meter 6 (power_meter.kicad_sch)
- added sheet Power channel 1 (lm5190.kicad_sch)
- added sheet Power channel 2 (lm5190.kicad_sch)
- note added: "Zdroj RIDEN RD-800-68"
- company: (none) -> David Haisman
- title: (none) -> ${PROJECTNAME}
- moved on the sheet: J101, J102, J103, J104, R101, R102
