File: PCB_design/Power_unit/Power_unit_A1/auxiliary_power_supply.kicad_sch (KiCad schematic)
At the start: 39 parts, among them U1501 TPS7A4101DGN, U1502 LM27761, U1503 TPS54360BQDDARQ1, U1504 TPS54360BQDDARQ1

Commit message: Initial thesis release
Parts:
- renumbered C1501 to C201, C1502 to C202, C1503 to C203, C1504 to C204, C1505 to C205, C1506 to C206, C1507 to C207, C1508 to C208, C1509 to C209, C1510 to C210, C1511 to C211, C1512 to C212, C1513 to C213, C1514 to C214, C1515 to C215, C1516 to C216, C1517 to C217, C1518 to C218, C1519 to C219, D1501 to D201, D1502 to D202, L1501 to L201, L1502 to L202, R1501 to R201, R1502 to R202, R1503 to R203, R1504 to R204, R1505 to R205, R1506 to R206, R1507 to R207, R1508 to R208, R1509 to R209, R1510 to R210, R1511 to R211, R1512 to R212, U1501 to U201, U1502 to U202, U1503 to U203, U1504 to U204
Connections:
- net +3V3: no longer C201.1, U202.1 (VIN), U202.6 (EN)
- net +48V renamed V_{IN}
- new net +3.3V: C201.1, U202.1 (VIN), U202.6 (EN)

Commit message: WIP
Parts:
- removed C204, C212: 10u, symbol Device:C
- removed C210: 10n, symbol Device:C
- removed R205: 100k, symbol Device:R
- removed R206: 11k, symbol Device:R
- removed U201: TPS7A4101DGN, Package_SO:Texas_DGN0008B_VSSOP-8-1EP_3x3mm_P0.65mm_EP2x3mm_Mask1.88x1.98mm_ThermalVias, symbol Regulator_Linear:TPS7A4101DGN
- C201, C202, C203, C205, C206, C207, C208, C209, C211, C213, C214, C215, C216, C217: symbol Device:C -> Device:C_Small
Connections:
- net +3.3V: no longer C201.1
- net +3V3: no longer C216.1
- net +5V: no longer C217.1
- net -5V: no longer C213.1
- net GND: no longer C201.2, C202.2, C203.2, C206.2, C207.2, C208.2, C209.2, C211.2, C213.2, C216.2, C217.2
- net V_{IN}: no longer C202.1, C203.1
- net at C205.1: no longer U202.8 (C+)
- net at C205.2: no longer U202.7 (C-)
- net at U203.1 (BOOT): no longer C214.2
- net at R201.1, U203.6 (COMP): no longer C208.1
- net at D201.1 (K), L201.2, U203.8 (SW): no longer C214.1
- net at R202.1, U204.6 (COMP): no longer C209.1
- net at C206.1: no longer R201.2
- net at D202.1 (K), L202.2, U204.8 (SW): no longer C215.1
- net at U204.1 (BOOT): no longer C215.2
- net at U202.3 (CPOUT): no longer C211.1
- net at R202.2: no longer C207.1
Other:
- company: (none) -> David Haisman
- title: Power supply - low level driver -> ${PROJECTNAME}
