File: PCB_design/Power_unit/Power_unit_A1/channel_enable.kicad_sch (KiCad schematic)
At the start: 6 parts, among them Q501 Q_NPN_EBC, Q502 PMOS

Commit message: Initial thesis release
Parts:
- removed D501: ?12V, symbol Device:D_Zener
- removed Q501: Q_NPN_EBC, symbol Device:Q_NPN_EBC
- removed Q502: PMOS, symbol Simulation_SPICE:PMOS
- removed R501: 100k, symbol Device:R
- removed R502: 10k, symbol Device:R
- removed R503: R, symbol Device:R
- added D1101: ?12V, symbol Device:D_Zener
- added Q1101: Q_NPN_EBC, symbol Device:Q_NPN_EBC
- added Q1102: PMOS, symbol Simulation_SPICE:PMOS
- added R1101: 100k, symbol Device:R
- added R1102: 10k, symbol Device:R
- added R1103: 1k, symbol Device:R
Connections:
- net -5V: now also Q1101.1 (E)
- net EN: now also R1102.1
- net V_{IN}: now also D1101.1 (K), Q1102.3 (S), R1101.1
- net V_{out}: now also Q1102.1 (D)
- new net: Q1101.2 (B), R1102.2
- new net: D1101.2 (A), Q1102.2 (G), R1101.2, R1103.1
- new net: Q1101.3 (C), R1103.2
Other:
- title: Power supply - low level driver -> (none)

Commit message: WIP
Parts:
- renumbered D1101 to D601, Q1102 to Q601, Q1101 to Q602, R1101 to R601, R1103 to R602, R1102 to R603
Other:
- company: (none) -> David Haisman
- title: (none) -> ${PROJECTNAME}
Changed lines of the file:
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@@
 	(generator_version "9.0")
 	(paper "A4")
+	(title_block
+		(title "${PROJECTNAME}")
+		(date "2025-11-22")
+		(rev "A.1")
+		(company "David Haisman")
+	)
 	(junction
 		(at 124.46 82.55)
@@
 		(on_board yes)
 		(dnp no)
-		(property "Reference" "R1102"
+		(property "Reference" "R603"
 			(at 137.16 109.474 90)
 			(effects
@@
 		(instances
 			(project "Power_unit_A1"
+				(path "/39e95423-af83-4645-98fc-4a660ba074aa/255bc17f-f051-4e1e-a239-9dca5da3a160"
+					(reference "R2003")
+					(unit 1)
+				)
+				(path "/39e95423-af83-4645-98fc-4a660ba074aa/6f700a06-8d8f-41dc-b772-46943792089e"
+					(reference "R1903")
+					(unit 1)
+				)
 				(path "/39e95423-af83-4645-98fc-4a660ba074aa/818a02ce-012a-459a-87bd-7e045ee7c385"
 					(reference "R1702")
@@
 				(path "/39e95423-af83-4645-98fc-4a660ba074aa/d722fe20-a3af-4c71-bd36-1af3ea59cbb5"
 					(reference "R1102")
+					(unit 1)
+				)
+				(path "/39e95423-af83-4645-98fc-4a660ba074aa/ebc2faa2-7b0f-4ce2-b085-cd3b9b2e7c96"
+					(reference "R603")
 					(unit 1)
 				)
@@
 		(dnp no)
 		(fields_autoplaced yes)
-		(property "Reference" "R1101"
+		(property "Reference" "R601"
 			(at 127 86.3599 0)
 			(effects
@@
 		(instances
 			(project "Power_unit_A1"
+				(path "/39e95423-af83-4645-98fc-4a660ba074aa/255bc17f-f051-4e1e-a239-9dca5da3a160"
+					(reference "R2001")
+					(unit 1)
+				)
+				(path "/39e95423-af83-4645-98fc-4a660ba074aa/6f700a06-8d8f-41dc-b772-46943792089e"
+					(reference "R1901")
+					(unit 1)
+				)
 				(path "/39e95423-af83-4645-98fc-4a660ba074aa/818a02ce-012a-459a-87bd-7e045ee7c385"
 					(reference "R1701")
@@
 				(path "/39e95423-af83-4645-98fc-4a660ba074aa/d722fe20-a3af-4c71-bd36-1af3ea59cbb5"
 					(reference "R1101")
+					(unit 1)
+				)
+				(path "/39e95423-af83-4645-98fc-4a660ba074aa/ebc2faa2-7b0f-4ce2-b085-cd3b9b2e7c96"
+					(reference "R601")
 					(unit 1)
 				)
@@
 		(dnp no)
 		(fields_autoplaced yes)
-		(property "Reference" "R1103"
+		(property "Reference" "R602"
 			(at 152.4 100.3299 0)
 			(effects
@@
 		(instances
 			(project "Power_unit_A1"
+				(path "/39e95423-af83-4645-98fc-4a660ba074aa/255bc17f-f051-4e1e-a239-9dca5da3a160"
+					(reference "R2002")
+					(unit 1)
+				)
+				(path "/39e95423-af83-4645-98fc-4a660ba074aa/6f700a06-8d8f-41dc-b772-46943792089e"
+					(reference "R1902")
+					(unit 1)
+				)
 				(path "/39e95423-af83-4645-98fc-4a660ba074aa/818a02ce-012a-459a-87bd-7e045ee7c385"
 					(reference "R1703")
@@
 				(path "/39e95423-af83-4645-98fc-4a660ba074aa/d722fe20-a3af-4c71-bd36-1af3ea59cbb5"
 					(reference "R1103")
+					(unit 1)
+				)
+				(path "/39e95423-af83-4645-98fc-4a660ba074aa/ebc2faa2-7b0f-4ce2-b085-cd3b9b2e7c96"
+					(reference "R602")
 					(unit 1)
 				)
@@
 		(on_board yes)
 		(dnp no)
-		(property "Reference" "Q1102"
+		(property "Reference" "Q601"
 			(at 149.86 76.2 90)
 			(effects
@@
 		(instances
 			(project "Power_unit_A1"
+				(path "/39e95423-af83-4645-98fc-4a660ba074aa/255bc17f-f051-4e1e-a239-9dca5da3a160"
+					(reference "Q2001")
+					(unit 1)
+				)
+				(path "/39e95423-af83-4645-98fc-4a660ba074aa/6f700a06-8d8f-41dc-b772-46943792089e"
+					(reference "Q1901")
+					(unit 1)
+				)
 				(path "/39e95423-af83-4645-98fc-4a660ba074aa/818a02ce-012a-459a-87bd-7e045ee7c385"
 					(reference "Q1702")
@@
 				(path "/39e95423-af83-4645-98fc-4a660ba074aa/d722fe20-a3af-4c71-bd36-1af3ea59cbb5"
 					(reference "Q1102")
+					(unit 1)
+				)
+				(path "/39e95423-af83-4645-98fc-4a660ba074aa/ebc2faa2-7b0f-4ce2-b085-cd3b9b2e7c96"
+					(reference "Q601")
 					(unit 1)
 				)
@@
 		(dnp no)
 		(fields_autoplaced yes)
-		(property "Reference" "Q1101"
+		(property "Reference" "Q602"
 			(at 152.4 110.4899 0)
 			(effects
@@
 		(instances
 			(project "Power_unit_A1"
+				(path "/39e95423-af83-4645-98fc-4a660ba074aa/255bc17f-f051-4e1e-a239-9dca5da3a160"
+					(reference "Q2002")
+					(unit 1)
+				)
+				(path "/39e95423-af83-4645-98fc-4a660ba074aa/6f700a06-8d8f-41dc-b772-46943792089e"
+					(reference "Q1902")
+					(unit 1)
+				)
 				(path "/39e95423-af83-4645-98fc-4a660ba074aa/818a02ce-012a-459a-87bd-7e045ee7c385"
 					(reference "Q1701")
@@
 				(path "/39e95423-af83-4645-98fc-4a660ba074aa/d722fe20-a3af-4c71-bd36-1af3ea59cbb5"
 					(reference "Q1101")
+					(unit 1)
+				)
+				(path "/39e95423-af83-4645-98fc-4a660ba074aa/ebc2faa2-7b0f-4ce2-b085-cd3b9b2e7c96"
+					(reference "Q602")
 					(unit 1)
 				)
@@
 		(dnp no)
 		(fields_autoplaced yes)
-		(property "Reference" "#PWR01101"
+		(property "Reference" "#PWR0601"
 			(at 149.86 114.3 0)
 			(effects
@@
 		(instances
 			(project "Power_unit_A1"
+				(path "/39e95423-af83-4645-98fc-4a660ba074aa/255bc17f-f051-4e1e-a239-9dca5da3a160"
+					(reference "#PWR02001")
+					(unit 1)
+				)
+				(path "/39e95423-af83-4645-98fc-4a660ba074aa/6f700a06-8d8f-41dc-b772-46943792089e"
+					(reference "#PWR01901")
+					(unit 1)
+				)
 				(path "/39e95423-af83-4645-98fc-4a660ba074aa/818a02ce-012a-459a-87bd-7e045ee7c385"
 					(reference "#PWR01701")
@@
 				(path "/39e95423-af83-4645-98fc-4a660ba074aa/d722fe20-a3af-4c71-bd36-1af3ea59cbb5"
 					(reference "#PWR01101")
+					(unit 1)
+				)
+				(path "/39e95423-af83-4645-98fc-4a660ba074aa/ebc2faa2-7b0f-4ce2-b085-cd3b9b2e7c96"
+					(reference "#PWR0601")
 					(unit 1)
 				)
@@
 		(dnp no)
 		(fields_autoplaced yes)
-		(property "Reference" "D1101"
+		(property "Reference" "D601"
 			(at 137.16 86.3599 90)
 			(effects
@@
 		(instances
 			(project "Power_unit_A1"
+				(path "/39e95423-af83-4645-98fc-4a660ba074aa/255bc17f-f051-4e1e-a239-9dca5da3a160"
+					(reference "D2001")
+					(unit 1)
+				)
+				(path "/39e95423-af83-4645-98fc-4a660ba074aa/6f700a06-8d8f-41dc-b772-46943792089e"
+					(reference "D1901")
+					(unit 1)
+				)
 				(path "/39e95423-af83-4645-98fc-4a660ba074aa/818a02ce-012a-459a-87bd-7e045ee7c385"
 					(reference "D1701")
@@
 					(unit 1)
 				)
+				(path "/39e95423-af83-4645-98fc-4a660ba074aa/ebc2faa2-7b0f-4ce2-b085-cd3b9b2e7c96"
+					(reference "D601")
+					(unit 1)
+				)
