File: PCB_design/Power_unit/Power_unit_A1/filter_input.kicad_sch (KiCad schematic)
At the start: 1 part

Commit message: Initial thesis release
Parts:
- removed C1101: C, symbol Device:C
- added C901: C, symbol Device:C
Connections:
- net GND: now also C901.2
- new net OUT: C901.1
Changed lines of the file:
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@@
 		(date "2024-06-28")
-	)
-	(junction
-		(at 187.96 91.44)
-		(diameter 0)
-		(color 0 0 0 0)
 	)
 	(wire
 		(pts
-			(xy 187.96 91.44) (xy 209.55 91.44)
+			(xy 153.67 87.63) (xy 176.53 87.63)
 		)
 		(stroke
@@
 	(wire
 		(pts
-			(xy 187.96 91.44) (xy 187.96 95.25)
+			(xy 153.67 87.63) (xy 153.67 91.44)
 		)
 		(stroke
@@
 	(wire
 		(pts
-			(xy 83.82 91.44) (xy 187.96 91.44)
+			(xy 50.8 87.63) (xy 60.96 87.63)
 		)
 		(stroke
@@
 	(hierarchical_label "IN"
 		(shape input)
-		(at 83.82 91.44 180)
+		(at 50.8 87.63 180)
 		(effects
 			(font
@@
 	(hierarchical_label "OUT"
 		(shape output)
-		(at 209.55 91.44 0)
+		(at 176.53 87.63 0)
 		(effects
 			(font
@@
 	)
 	(symbol
+		(lib_id "power:GND")
+		(at 153.67 99.06 0)
+		(unit 1)
+		(exclude_from_sim no)
+		(in_bom yes)
+		(on_board yes)
+		(dnp no)
+		(property "Reference" "#PWR0901"
+			(at 153.67 105.41 0)
+			(effects
+				(font
+					(size 1.27 1.27)
+				)
+				(hide yes)
+			)
+		)
+		(property "Value" "GND"
+			(at 157.226 101.092 0)
+			(effects
+				(font
+					(size 1.27 1.27)
+				)
+			)
+		)
+		(property "Footprint" ""
+			(at 153.67 99.06 0)
+			(effects
+				(font
+					(size 1.27 1.27)
+				)
+				(hide yes)
+			)
+		)
+		(property "Datasheet" ""
+			(at 153.67 99.06 0)
+			(effects
+				(font
+					(size 1.27 1.27)
+				)
+				(hide yes)
+			)
+		)
+		(property "Description" "Power symbol creates a global label with name \"GND\" , ground"
+			(at 153.67 99.06 0)
+			(effects
+				(font
+					(size 1.27 1.27)
+				)
+				(hide yes)
+			)
+		)
+		(pin "1"
+		)
+		(instances
+			(project "Low-level-driver"
+				(path "/2e43a8c9-1b23-4896-a481-133b23afb346/fc16a9b7-58fe-46ae-b1a6-53c2dcbd67dc"
+					(reference "#PWR01001")
+					(unit 1)
+				)
+			)
+			(project "Low-level-driver"
+				(path "/39e95423-af83-4645-98fc-4a660ba074aa/45b56bb9-b346-4ff4-8959-e298f8ce3eca"
+					(reference "#PWR0901")
+					(unit 1)
+				)
+			)
+		)
+	)
+	(symbol
 		(lib_id "Device:C")
-		(at 187.96 99.06 0)
+		(at 153.67 95.25 0)
 		(unit 1)
 		(exclude_from_sim no)
@@
 		(dnp no)
 		(fields_autoplaced yes)
-		(property "Reference" "C1101"
-			(at 191.77 97.7899 0)
+		(property "Reference" "C901"
+			(at 157.48 93.9799 0)
 			(effects
 				(font
@@
 		)
 		(property "Value" "C"
-			(at 191.77 100.3299 0)
+			(at 157.48 96.5199 0)
 			(effects
 				(font
@@
 		)
 		(property "Footprint" ""
-			(at 188.9252 102.87 0)
+			(at 154.6352 99.06 0)
 			(effects
 				(font
@@
 		)
 		(property "Datasheet" "~"
-			(at 187.96 99.06 0)
+			(at 153.67 95.25 0)
 			(effects
 				(font
@@
 		)
 		(property "Description" "Unpolarized capacitor"
-			(at 187.96 99.06 0)
+			(at 153.67 95.25 0)
 			(effects
 				(font
@@
 		(instances
 			(project "Low-level-driver"
-				(path "/2e43a8c9-1b23-4896-a481-133b23afb346/7a6cc648-2320-4c5a-8776-ce46b8832613"
-					(reference "C1201")
-					(unit 1)
-				)
-				(path "/2e43a8c9-1b23-4896-a481-133b23afb346/a606a429-17db-405f-9eaf-8fc6a9c822cc"
-					(reference "C1101")
+				(path "/2e43a8c9-1b23-4896-a481-133b23afb346/fc16a9b7-58fe-46ae-b1a6-53c2dcbd67dc"
+					(reference "C1001")
 					(unit 1)
 				)
 			)
-		)
-	)
-	(symbol
-		(lib_id "power:GND")
-		(at 187.96 102.87 0)
-		(unit 1)
-		(exclude_from_sim no)
-		(in_bom yes)
-		(on_board yes)
-		(dnp no)
-		(property "Reference" "#PWR01101"
-			(at 187.96 109.22 0)
-			(effects
-				(font
-					(size 1.27 1.27)
-				)
-				(hide yes)
-			)
-		)
-		(property "Value" "GND"
-			(at 191.516 104.902 0)
-			(effects
-				(font
-					(size 1.27 1.27)
-				)
-			)
-		)
-		(property "Footprint" ""
-			(at 187.96 102.87 0)
-			(effects
-				(font
-					(size 1.27 1.27)
-				)
-				(hide yes)
-			)
-		)
-		(property "Datasheet" ""
-			(at 187.96 102.87 0)
-			(effects
-				(font
-					(size 1.27 1.27)
-				)
-				(hide yes)
-			)
-		)
-		(property "Description" "Power symbol creates a global label with name \"GND\" , ground"
-			(at 187.96 102.87 0)
-			(effects
-				(font
-					(size 1.27 1.27)
-				)
-				(hide yes)
-			)
-		)
-		(pin "1"
-		)
-		(instances
 			(project "Low-level-driver"
-				(path "/2e43a8c9-1b23-4896-a481-133b23afb346/7a6cc648-2320-4c5a-8776-ce46b8832613"
-					(reference "#PWR01201")
+				(path "/39e95423-af83-4645-98fc-4a660ba074aa/45b56bb9-b346-4ff4-8959-e298f8ce3eca"
+					(reference "C901")
 					(unit 1)
 				)
-				(path "/2e43a8c9-1b23-4896-a481-133b23afb346/a606a429-17db-405f-9eaf-8fc6a9c822cc"
-					(reference "#PWR01101")
-					(unit 1)
-				)

Commit message: WIP
Parts:
- C1001: renamed from C901; symbol Device:C -> Device:C_Small
Connections:
- net GND: no longer C1001.2
- net OUT: no longer C1001.1
Other:
- company: (none) -> David Haisman
- title: Power supply - low level driver -> ${PROJECTNAME}
Changed lines of the file:
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@@
 	(paper "A4")
 	(title_block
-		(title "Power supply - low level driver")
-		(date "2024-06-28")
+		(title "${PROJECTNAME}")
+		(date "2025-11-22")
+		(rev "A.1")
+		(company "David Haisman")
 	)
 	(wire
@@
 		(on_board yes)
 		(dnp no)
-		(property "Reference" "#PWR0901"
+		(property "Reference" "#PWR01001"
 			(at 153.67 105.41 0)
 			(effects
@@
 		)
 		(instances
-			(project "Low-level-driver"
-				(path "/2e43a8c9-1b23-4896-a481-133b23afb346/fc16a9b7-58fe-46ae-b1a6-53c2dcbd67dc"
+			(project ""
+				(path "/39e95423-af83-4645-98fc-4a660ba074aa/45b56bb9-b346-4ff4-8959-e298f8ce3eca"
 					(reference "#PWR01001")
 					(unit 1)
 				)
-			)
-			(project "Low-level-driver"
-				(path "/39e95423-af83-4645-98fc-4a660ba074aa/45b56bb9-b346-4ff4-8959-e298f8ce3eca"
-					(reference "#PWR0901")
+				(path "/39e95423-af83-4645-98fc-4a660ba074aa/d11ff0cf-1c79-477c-af91-4785ea35734b"
+					(reference "#PWR02501")
 					(unit 1)
 				)
@@
 	)
 	(symbol
-		(lib_id "Device:C")
+		(lib_id "Device:C_Small")
 		(at 153.67 95.25 0)
 		(unit 1)
@@
 		(dnp no)
 		(fields_autoplaced yes)
-		(property "Reference" "C901"
-			(at 157.48 93.9799 0)
+		(property "Reference" "C1001"
+			(at 156.21 93.9862 0)
 			(effects
 				(font
@@
 		)
 		(property "Value" "C"
-			(at 157.48 96.5199 0)
+			(at 156.21 96.5262 0)
 			(effects
 				(font
@@
 		)
 		(property "Footprint" ""
-			(at 154.6352 99.06 0)
+			(at 153.67 95.25 0)
 			(effects
 				(font
@@
 			)
 		)
-		(property "Description" "Unpolarized capacitor"
+		(property "Description" "Unpolarized capacitor, small symbol"
 			(at 153.67 95.25 0)
 			(effects
@@
 		)
 		(instances
-			(project "Low-level-driver"
-				(path "/2e43a8c9-1b23-4896-a481-133b23afb346/fc16a9b7-58fe-46ae-b1a6-53c2dcbd67dc"
+			(project ""
+				(path "/39e95423-af83-4645-98fc-4a660ba074aa/45b56bb9-b346-4ff4-8959-e298f8ce3eca"
 					(reference "C1001")
 					(unit 1)
 				)
-			)
-			(project "Low-level-driver"
-				(path "/39e95423-af83-4645-98fc-4a660ba074aa/45b56bb9-b346-4ff4-8959-e298f8ce3eca"
-					(reference "C901")
+				(path "/39e95423-af83-4645-98fc-4a660ba074aa/d11ff0cf-1c79-477c-af91-4785ea35734b"
+					(reference "C2501")
 					(unit 1)
 				)
