File: PCB_design/Power_unit/Power_unit_A1/filter_output.kicad_sch (KiCad schematic)
At the start: 1 part

Commit message: Initial thesis release
Parts:
- renumbered C1101 to C701
Changed lines of the file:
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@@
 		(dnp no)
 		(fields_autoplaced yes)
-		(property "Reference" "C1101"
+		(property "Reference" "C701"
 			(at 191.77 97.7899 0)
 			(effects
@@
 				)
 			)
+			(project "Low-level-driver"
+				(path "/39e95423-af83-4645-98fc-4a660ba074aa/20cf9902-7d32-4984-b311-7ec20afcd44b"
+					(reference "C701")
+					(unit 1)
+				)
+				(path "/39e95423-af83-4645-98fc-4a660ba074aa/7f5a6bae-77cc-49f4-bbf3-c2e71110d959"
+					(reference "C801")
+					(unit 1)
+				)
+			)
 		)
 	)
@@
 		(on_board yes)
 		(dnp no)
-		(property "Reference" "#PWR01101"
+		(property "Reference" "#PWR0701"
 			(at 187.96 109.22 0)
 			(effects
@@
 					(unit 1)
 				)
+			)
+			(project "Low-level-driver"
+				(path "/39e95423-af83-4645-98fc-4a660ba074aa/20cf9902-7d32-4984-b311-7ec20afcd44b"
+					(reference "#PWR0701")
+					(unit 1)
+				)
+				(path "/39e95423-af83-4645-98fc-4a660ba074aa/7f5a6bae-77cc-49f4-bbf3-c2e71110d959"
+					(reference "#PWR0801")
+					(unit 1)
+				)

Commit message: WIP
Parts:
- C801: renamed from C701; symbol Device:C -> Device:C_Small
Connections:
- net GND: no longer C801.2
- net IN: no longer C801.1
Other:
- company: (none) -> David Haisman
- title: Power supply - low level driver -> ${PROJECTNAME}
Changed lines of the file:
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@@
 	(paper "A4")
 	(title_block
-		(title "Power supply - low level driver")
-		(date "2024-06-28")
+		(title "${PROJECTNAME}")
+		(date "2025-11-22")
+		(rev "A.1")
+		(company "David Haisman")
 	)
 	(junction
@@
 	)
 	(symbol
-		(lib_id "Device:C")
+		(lib_id "Device:C_Small")
 		(at 187.96 99.06 0)
 		(unit 1)
@@
 		(dnp no)
 		(fields_autoplaced yes)
-		(property "Reference" "C701"
-			(at 191.77 97.7899 0)
+		(property "Reference" "C801"
+			(at 190.5 97.7962 0)
 			(effects
 				(font
@@
 		)
 		(property "Value" "C"
-			(at 191.77 100.3299 0)
+			(at 190.5 100.3362 0)
 			(effects
 				(font
@@
 		)
 		(property "Footprint" ""
-			(at 188.9252 102.87 0)
+			(at 187.96 99.06 0)
 			(effects
 				(font
@@
 			)
 		)
-		(property "Description" "Unpolarized capacitor"
+		(property "Description" "Unpolarized capacitor, small symbol"
 			(at 187.96 99.06 0)
 			(effects
@@
 		)
 		(instances
-			(project "Low-level-driver"
-				(path "/2e43a8c9-1b23-4896-a481-133b23afb346/7a6cc648-2320-4c5a-8776-ce46b8832613"
-					(reference "C1201")
-					(unit 1)
-				)
-				(path "/2e43a8c9-1b23-4896-a481-133b23afb346/a606a429-17db-405f-9eaf-8fc6a9c822cc"
-					(reference "C1101")
-					(unit 1)
-				)
-			)
-			(project "Low-level-driver"
+			(project ""
 				(path "/39e95423-af83-4645-98fc-4a660ba074aa/20cf9902-7d32-4984-b311-7ec20afcd44b"
-					(reference "C701")
+					(reference "C801")
+					(unit 1)
+				)
+				(path "/39e95423-af83-4645-98fc-4a660ba074aa/380e1241-e27a-406c-8ff1-1cc9f5ff715e"
+					(reference "C2401")
 					(unit 1)
 				)
 				(path "/39e95423-af83-4645-98fc-4a660ba074aa/7f5a6bae-77cc-49f4-bbf3-c2e71110d959"
 					(reference "C801")
+					(unit 1)
+				)
+				(path "/39e95423-af83-4645-98fc-4a660ba074aa/a039f445-7ed4-4a1a-9ecd-1e141bc06e0f"
+					(reference "C2301")
 					(unit 1)
 				)
@@
 		(on_board yes)
 		(dnp no)
-		(property "Reference" "#PWR0701"
+		(property "Reference" "#PWR0801"
 			(at 187.96 109.22 0)
 			(effects
@@
 		)
 		(instances
-			(project "Low-level-driver"
-				(path "/2e43a8c9-1b23-4896-a481-133b23afb346/7a6cc648-2320-4c5a-8776-ce46b8832613"
-					(reference "#PWR01201")
-					(unit 1)
-				)
-				(path "/2e43a8c9-1b23-4896-a481-133b23afb346/a606a429-17db-405f-9eaf-8fc6a9c822cc"
-					(reference "#PWR01101")
-					(unit 1)
-				)
-			)
-			(project "Low-level-driver"
+			(project ""
 				(path "/39e95423-af83-4645-98fc-4a660ba074aa/20cf9902-7d32-4984-b311-7ec20afcd44b"
-					(reference "#PWR0701")
+					(reference "#PWR0801")
+					(unit 1)
+				)
+				(path "/39e95423-af83-4645-98fc-4a660ba074aa/380e1241-e27a-406c-8ff1-1cc9f5ff715e"
+					(reference "#PWR02401")
 					(unit 1)
 				)
@@
 					(unit 1)
 				)
+				(path "/39e95423-af83-4645-98fc-4a660ba074aa/a039f445-7ed4-4a1a-9ecd-1e141bc06e0f"
+					(reference "#PWR02301")
+					(unit 1)
+				)
