File: PCB_design/Power_unit/Power_unit_A1/gpio_expander.kicad_sch (KiCad schematic)
At the start: 3 parts, among them U1601 TCA9535PWR

Commit message: Initial thesis release
Parts:
- renumbered C1601 to C1001, R1601 to R1001, U1601 to U1001
Changed lines of the file:
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@@
 		)
 	)
-	(global_label "I^{2}C{SCL SDA}"
+	(hierarchical_label "P_{03}"
+		(shape bidirectional)
+		(at 165.1 82.55 0)
+		(effects
+			(font
+				(size 1.27 1.27)
+			)
+			(justify left)
+		)
+	)
+	(hierarchical_label "P_{13}"
+		(shape bidirectional)
+		(at 165.1 105.41 0)
+		(effects
+			(font
+				(size 1.27 1.27)
+			)
+			(justify left)
+		)
+	)
+	(hierarchical_label "P_{02}"
+		(shape bidirectional)
+		(at 165.1 80.01 0)
+		(effects
+			(font
+				(size 1.27 1.27)
+			)
+			(justify left)
+		)
+	)
+	(hierarchical_label "{I^{2}C}"
 		(shape input)
 		(at 121.92 63.5 180)
-		(fields_autoplaced yes)
 		(effects
 			(font
@@
 			)
 			(justify right)
-		)
-		(property "Intersheetrefs" "${INTERSHEET_REFS}"
-			(at 106.556 63.5 0)
-			(effects
-				(font
-					(size 1.27 1.27)
-				)
-				(justify right)
-				(hide yes)
-			)
-		)
-	)
-	(hierarchical_label "P_{03}"
-		(shape bidirectional)
-		(at 165.1 82.55 0)
-		(effects
-			(font
-				(size 1.27 1.27)
-			)
-			(justify left)
-		)
-	)
-	(hierarchical_label "P_{13}"
-		(shape bidirectional)
-		(at 165.1 105.41 0)
-		(effects
-			(font
-				(size 1.27 1.27)
-			)
-			(justify left)
-		)
-	)
-	(hierarchical_label "P_{02}"
-		(shape bidirectional)
-		(at 165.1 80.01 0)
-		(effects
-			(font
-				(size 1.27 1.27)
-			)
-			(justify left)
 		)
 	)
@@
 		(dnp no)
 		(fields_autoplaced yes)
-		(property "Reference" "#PWR01604"
+		(property "Reference" "#PWR01004"
 			(at 147.32 129.54 0)
 			(effects
@@
 		)
 		(instances
-			(project "Low-level-driver"
-				(path "/2e43a8c9-1b23-4896-a481-133b23afb346/741d97eb-4d41-46a3-bc95-8b959e917640"
-					(reference "#PWR01604")
+			(project "Power_unit_A1"
+				(path "/39e95423-af83-4645-98fc-4a660ba074aa/b2e8286b-01af-45a1-ab90-710a69d0a80f"
+					(reference "#PWR01004")
 					(unit 1)
 				)
@@
 		(on_board yes)
 		(dnp no)
-		(property "Reference" "#PWR01601"
+		(property "Reference" "#PWR01001"
 			(at 116.84 76.2 0)
 			(effects
@@
 		)
 		(instances
-			(project "Low-level-driver"
-				(path "/2e43a8c9-1b23-4896-a481-133b23afb346/741d97eb-4d41-46a3-bc95-8b959e917640"
-					(reference "#PWR01601")
+			(project "Power_unit_A1"
+				(path "/39e95423-af83-4645-98fc-4a660ba074aa/b2e8286b-01af-45a1-ab90-710a69d0a80f"
+					(reference "#PWR01001")
 					(unit 1)
 				)
@@
 		(on_board yes)
 		(dnp no)
-		(property "Reference" "#PWR01602"
+		(property "Reference" "#PWR01002"
 			(at 134.62 72.39 0)
 			(effects
@@
 		)
 		(instances
-			(project "Low-level-driver"
-				(path "/2e43a8c9-1b23-4896-a481-133b23afb346/741d97eb-4d41-46a3-bc95-8b959e917640"
-					(reference "#PWR01602")
+			(project "Power_unit_A1"
+				(path "/39e95423-af83-4645-98fc-4a660ba074aa/b2e8286b-01af-45a1-ab90-710a69d0a80f"
+					(reference "#PWR01002")
 					(unit 1)
 				)
@@
 		(dnp no)
 		(fields_autoplaced yes)
-		(property "Reference" "U1601"
+		(property "Reference" "U1001"
 			(at 149.5141 67.31 0)
 			(effects
@@
 		)
 		(instances
-			(project "Low-level-driver"
-				(path "/2e43a8c9-1b23-4896-a481-133b23afb346/741d97eb-4d41-46a3-bc95-8b959e917640"
-					(reference "U1601")
+			(project "Power_unit_A1"
+				(path "/39e95423-af83-4645-98fc-4a660ba074aa/b2e8286b-01af-45a1-ab90-710a69d0a80f"
+					(reference "U1001")
 					(unit 1)
 				)
@@
 		(on_board yes)
 		(dnp no)
-		(property "Reference" "R1601"
+		(property "Reference" "R1001"
 			(at 112.014 75.184 0)
 			(effects
@@
 		)
 		(instances
-			(project "Low-level-driver"
-				(path "/2e43a8c9-1b23-4896-a481-133b23afb346/741d97eb-4d41-46a3-bc95-8b959e917640"
-					(reference "R1601")
+			(project "Power_unit_A1"
+				(path "/39e95423-af83-4645-98fc-4a660ba074aa/b2e8286b-01af-45a1-ab90-710a69d0a80f"
+					(reference "R1001")
 					(unit 1)
 				)
@@
 		(on_board yes)
 		(dnp no)
-		(property "Reference" "#PWR01603"
+		(property "Reference" "#PWR01003"
 			(at 147.32 69.85 0)
 			(effects
@@
 		)
 		(instances
-			(project "Low-level-driver"
-				(path "/2e43a8c9-1b23-4896-a481-133b23afb346/741d97eb-4d41-46a3-bc95-8b959e917640"
-					(reference "#PWR01603")
+			(project "Power_unit_A1"
+				(path "/39e95423-af83-4645-98fc-4a660ba074aa/b2e8286b-01af-45a1-ab90-710a69d0a80f"
+					(reference "#PWR01003")
 					(unit 1)
 				)
@@
 		(on_board yes)
 		(dnp no)
-		(property "Reference" "C1601"
+		(property "Reference" "C1001"
 			(at 139.446 63.754 90)
 			(effects
@@
 		)
 		(instances
-			(project "Low-level-driver"
-				(path "/2e43a8c9-1b23-4896-a481-133b23afb346/741d97eb-4d41-46a3-bc95-8b959e917640"
-					(reference "C1601")
+			(project "Power_unit_A1"
+				(path "/39e95423-af83-4645-98fc-4a660ba074aa/b2e8286b-01af-45a1-ab90-710a69d0a80f"
+					(reference "C1001")
 					(unit 1)
 				)

Commit message: WIP
Parts:
- C1001: symbol Device:C -> Device:C_Small
Connections:
- net +3V3: no longer C1001.1
- net GND: no longer C1001.2
Other:
- company: (none) -> David Haisman
- title: Power supply - low level driver -> ${PROJECTNAME}
Changed lines of the file:
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@@
 	(paper "A4")
 	(title_block
-		(title "Power supply - low level driver")
-		(date "2024-06-28")
+		(title "${PROJECTNAME}")
+		(date "2025-11-22")
+		(rev "A.1")
+		(company "David Haisman")
 	)
 	(junction
@@
 	(junction
 		(at 147.32 123.19)
-		(diameter 0)
-		(color 0 0 0 0)
-	)
-	(junction
-		(at 147.32 66.04)
 		(diameter 0)
 		(color 0 0 0 0)
@@
 	)
 	(symbol
-		(lib_id "Device:C")
+		(lib_id "Device:C_Small")
 		(at 143.51 66.04 270)
 		(unit 1)
@@
 		)
 		(property "Footprint" ""
-			(at 139.7 67.0052 0)
+			(at 143.51 66.04 0)
 			(effects
 				(font
@@
 			)
 		)
-		(property "Description" "Unpolarized capacitor"
+		(property "Description" "Unpolarized capacitor, small symbol"
 			(at 143.51 66.04 0)
 			(effects
