File: PCB_design/Power_unit/Power_unit_A1/power_meter.kicad_sch (KiCad schematic)
At the start: 4 parts, among them U701 INA237

Commit message: Initial thesis release
Parts:
- renumbered NT702 to NT1301, NT701 to NT1302, R701 to R1301, U701 to U1301
Changed lines of the file:
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@@
 		)
 	)
-	(global_label "I^{2}C{SCL SDA}"
+	(hierarchical_label "{I^{2}C}"
 		(shape input)
 		(at 101.6 83.82 0)
-		(fields_autoplaced yes)
 		(effects
 			(font
@@
 			)
 			(justify left)
-		)
-		(property "Intersheetrefs" "${INTERSHEET_REFS}"
-			(at 116.964 83.82 0)
-			(effects
-				(font
-					(size 1.27 1.27)
-				)
-				(justify left)
-				(hide yes)
-			)
 		)
 	)
@@
 		(on_board yes)
 		(dnp no)
-		(property "Reference" "#PWR0702"
+		(property "Reference" "#PWR01302"
 			(at 74.93 114.3 0)
 			(effects
@@
 		)
 		(instances
-			(project "Low-level-driver"
-				(path "/2e43a8c9-1b23-4896-a481-133b23afb346/128e4573-9270-4dc9-a769-eeca3ba2582e"
-					(reference "#PWR0702")
-					(unit 1)
-				)
-				(path "/2e43a8c9-1b23-4896-a481-133b23afb346/427b1730-dc56-4e6c-8a7f-70a3ace5a196"
-					(reference "#PWR0802")
-					(unit 1)
-				)
-				(path "/2e43a8c9-1b23-4896-a481-133b23afb346/816f3957-0c05-4424-bbd1-ce08a032f88f"
-					(reference "#PWR0902")
+			(project "Power_unit_A1"
+				(path "/39e95423-af83-4645-98fc-4a660ba074aa/1fe5ab8d-eac1-482f-8e38-d7702b18d2e6"
+					(reference "#PWR01502")
+					(unit 1)
+				)
+				(path "/39e95423-af83-4645-98fc-4a660ba074aa/bd9c852b-3ca3-4af0-9c02-b6882fbbbc1b"
+					(reference "#PWR01302")
+					(unit 1)
+				)
+				(path "/39e95423-af83-4645-98fc-4a660ba074aa/c6b3704a-c3a9-40bb-8e0a-b29cf84caa9f"
+					(reference "#PWR01402")
 					(unit 1)
 				)
@@
 		(on_board yes)
 		(dnp no)
-		(property "Reference" "#PWR0701"
+		(property "Reference" "#PWR01301"
 			(at 74.93 86.36 0)
 			(effects
@@
 		)
 		(instances
-			(project "Low-level-driver"
-				(path "/2e43a8c9-1b23-4896-a481-133b23afb346/128e4573-9270-4dc9-a769-eeca3ba2582e"
-					(reference "#PWR0701")
-					(unit 1)
-				)
-				(path "/2e43a8c9-1b23-4896-a481-133b23afb346/427b1730-dc56-4e6c-8a7f-70a3ace5a196"
-					(reference "#PWR0801")
-					(unit 1)
-				)
-				(path "/2e43a8c9-1b23-4896-a481-133b23afb346/816f3957-0c05-4424-bbd1-ce08a032f88f"
-					(reference "#PWR0901")
+			(project "Power_unit_A1"
+				(path "/39e95423-af83-4645-98fc-4a660ba074aa/1fe5ab8d-eac1-482f-8e38-d7702b18d2e6"
+					(reference "#PWR01501")
+					(unit 1)
+				)
+				(path "/39e95423-af83-4645-98fc-4a660ba074aa/bd9c852b-3ca3-4af0-9c02-b6882fbbbc1b"
+					(reference "#PWR01301")
+					(unit 1)
+				)
+				(path "/39e95423-af83-4645-98fc-4a660ba074aa/c6b3704a-c3a9-40bb-8e0a-b29cf84caa9f"
+					(reference "#PWR01401")
 					(unit 1)
 				)
@@
 		(on_board yes)
 		(dnp no)
-		(property "Reference" "NT701"
+		(property "Reference" "NT1302"
 			(at 55.372 104.902 0)
 			(effects
@@
 		)
 		(instances
-			(project "Low-level-driver"
-				(path "/2e43a8c9-1b23-4896-a481-133b23afb346/128e4573-9270-4dc9-a769-eeca3ba2582e"
-					(reference "NT701")
-					(unit 1)
-				)
-				(path "/2e43a8c9-1b23-4896-a481-133b23afb346/427b1730-dc56-4e6c-8a7f-70a3ace5a196"
-					(reference "NT801")
-					(unit 1)
-				)
-				(path "/2e43a8c9-1b23-4896-a481-133b23afb346/816f3957-0c05-4424-bbd1-ce08a032f88f"
-					(reference "NT901")
+			(project "Power_unit_A1"
+				(path "/39e95423-af83-4645-98fc-4a660ba074aa/1fe5ab8d-eac1-482f-8e38-d7702b18d2e6"
+					(reference "NT1502")
+					(unit 1)
+				)
+				(path "/39e95423-af83-4645-98fc-4a660ba074aa/bd9c852b-3ca3-4af0-9c02-b6882fbbbc1b"
+					(reference "NT1302")
+					(unit 1)
+				)
+				(path "/39e95423-af83-4645-98fc-4a660ba074aa/c6b3704a-c3a9-40bb-8e0a-b29cf84caa9f"
+					(reference "NT1402")
 					(unit 1)
 				)
@@
 		(on_board yes)
 		(dnp no)
-		(property "Reference" "R701"
+		(property "Reference" "R1301"
 			(at 52.07 97.7899 0)
 			(effects
@@
 		)
 		(instances
-			(project "Low-level-driver"
-				(path "/2e43a8c9-1b23-4896-a481-133b23afb346/128e4573-9270-4dc9-a769-eeca3ba2582e"
-					(reference "R701")
-					(unit 1)
-				)
-				(path "/2e43a8c9-1b23-4896-a481-133b23afb346/427b1730-dc56-4e6c-8a7f-70a3ace5a196"
-					(reference "R801")
-					(unit 1)
-				)
-				(path "/2e43a8c9-1b23-4896-a481-133b23afb346/816f3957-0c05-4424-bbd1-ce08a032f88f"
-					(reference "R901")
+			(project "Power_unit_A1"
+				(path "/39e95423-af83-4645-98fc-4a660ba074aa/1fe5ab8d-eac1-482f-8e38-d7702b18d2e6"
+					(reference "R1501")
+					(unit 1)
+				)
+				(path "/39e95423-af83-4645-98fc-4a660ba074aa/bd9c852b-3ca3-4af0-9c02-b6882fbbbc1b"
+					(reference "R1301")
+					(unit 1)
+				)
+				(path "/39e95423-af83-4645-98fc-4a660ba074aa/c6b3704a-c3a9-40bb-8e0a-b29cf84caa9f"
+					(reference "R1401")
 					(unit 1)
 				)
@@
 		(on_board yes)
 		(dnp no)
-		(property "Reference" "NT702"
+		(property "Reference" "NT1301"
 			(at 55.88 93.726 0)
 			(effects
@@
 		)
 		(instances
-			(project "Low-level-driver"
-				(path "/2e43a8c9-1b23-4896-a481-133b23afb346/128e4573-9270-4dc9-a769-eeca3ba2582e"
-					(reference "NT702")
-					(unit 1)
-				)
-				(path "/2e43a8c9-1b23-4896-a481-133b23afb346/427b1730-dc56-4e6c-8a7f-70a3ace5a196"
-					(reference "NT802")
-					(unit 1)
-				)
-				(path "/2e43a8c9-1b23-4896-a481-133b23afb346/816f3957-0c05-4424-bbd1-ce08a032f88f"
-					(reference "NT902")
+			(project "Power_unit_A1"
+				(path "/39e95423-af83-4645-98fc-4a660ba074aa/1fe5ab8d-eac1-482f-8e38-d7702b18d2e6"
+					(reference "NT1501")
+					(unit 1)
+				)
+				(path "/39e95423-af83-4645-98fc-4a660ba074aa/bd9c852b-3ca3-4af0-9c02-b6882fbbbc1b"
+					(reference "NT1301")
+					(unit 1)
+				)
+				(path "/39e95423-af83-4645-98fc-4a660ba074aa/c6b3704a-c3a9-40bb-8e0a-b29cf84caa9f"
+					(reference "NT1401")
 					(unit 1)
 				)
@@
 		(dnp no)
 		(fields_autoplaced yes)
-		(property "Reference" "U701"
+		(property "Reference" "U1301"
 			(at 77.1241 80.01 0)
 			(effects
@@
 		)
 		(instances
-			(project "Low-level-driver"
-				(path "/2e43a8c9-1b23-4896-a481-133b23afb346/128e4573-9270-4dc9-a769-eeca3ba2582e"
-					(reference "U701")
-					(unit 1)
-				)
-				(path "/2e43a8c9-1b23-4896-a481-133b23afb346/427b1730-dc56-4e6c-8a7f-70a3ace5a196"
-					(reference "U801")
-					(unit 1)
-				)
-				(path "/2e43a8c9-1b23-4896-a481-133b23afb346/816f3957-0c05-4424-bbd1-ce08a032f88f"
-					(reference "U901")
-					(unit 1)
-				)
+			(project "Power_unit_A1"
+				(path "/39e95423-af83-4645-98fc-4a660ba074aa/1fe5ab8d-eac1-482f-8e38-d7702b18d2e6"
+					(reference "U1501")
+					(unit 1)
+				)
+				(path "/39e95423-af83-4645-98fc-4a660ba074aa/bd9c852b-3ca3-4af0-9c02-b6882fbbbc1b"
+					(reference "U1301")
+					(unit 1)
+				)
+				(path "/39e95423-af83-4645-98fc-4a660ba074aa/c6b3704a-c3a9-40bb-8e0a-b29cf84caa9f"
+					(reference "U1401")
+					(unit 1)
+				)

Commit message: WIP
Parts:
- removed NT1301, NT1302: NetTie_2, symbol Device:NetTie_2
- removed R1301: R, symbol Device:R
- added C2801: C_Small, symbol Device:C_Small
- added R2801, R2803: R_Small, symbol Device:R_Small
- added R2802: R_Shunt, symbol Device:R_Shunt
Connections:
- net V_{IN}: now also R2802.1; no longer U1301.8 (Vbus)
- net V_{OUT}: now also U1301.8 (Vbus), R2802.4
- net at U1301.9 (Vin-): now also C2801.2, R2803.2
- net at U1301.10 (Vin+): now also C2801.1, R2801.2
- net A0 renamed A_{0}
- net A1 renamed A_{1}
- new net: R2801.1, R2802.2
- new net: R2802.3, R2803.1
Other:
- company: (none) -> David Haisman
- title: Power supply - low level driver -> ${PROJECTNAME}
- moved on the sheet: U1301
