File: PCB_design/Power_unit/Power_unit_A1/power_supply.kicad_sch (KiCad schematic)
At the start: 39 parts, among them Q201 NMOS, Q202 NMOS, Q203 NMOS, Q204 NMOS, Q205 PMOS, Q206 Q_NPN_BCE, U201 LM5143

Commit message: Initial thesis release
Parts:
- removed Q205: PMOS, symbol Simulation_SPICE:PMOS
- removed Q206: Q_NPN_BCE, symbol Device:Q_NPN_BCE
- removed R209: 100k, symbol Device:R
- removed R210: 10k, symbol Device:R
- renumbered C214 to C1601, C213 to C1602, C215 to C1603, C201 to C1604, C202 to C1605, C203 to C1606, C204 to C1607, C205 to C1608, C206 to C1609, C207 to C1610, C208 to C1611, C209 to C1612, C210 to C1613, C211 to C1614, C212 to C1615, C218 to C1616, C217 to C1617, C216 to C1618, D201 to D1601, D202 to D1602, L201 to L1601, L202 to L1602, Q201 to Q1601, Q202 to Q1602, Q203 to Q1603, Q204 to Q1604, R201 to R1601, R202 to R1602, R203 to R1603, R204 to R1604, R205 to R1605, R206 to R1606, R207 to R1607, R208 to R1608, U201 to U1601
Connections:
- net Input: now also Q1601.1 (D), Q1603.1 (D), U1601.25 (VIN)
- net +3V3 renamed +3.3V
Other:
- title: Power supply - low level driver -> (none)

Commit message: WIP
Parts:
- removed C1601, C1602, C1603, C1604, C1605, C1606: C, symbol Device:C
- removed C1607: 0.1uF, symbol Device:C
- removed D1601: D_Schottky, symbol Device:D_Schottky
- removed L1601: L, symbol Device:L
- removed Q1601, Q1602: NMOS, symbol Simulation_SPICE:NMOS
- removed R1601, R1603, R1604: R, symbol Device:R
- removed R1602: 10k, symbol Device:R
- added R3: 10k, symbol Device:R
- C1608, C1609, C1610, C1611, C1612, C1613, C1614, C1615, C1616, C1617, C1618: symbol Device:C -> Device:C_Small
Connections:
- net +3.3V: now also R3.2
- net GND: no longer C1608.2, C1609.2, C1610.2, C1611.1, C1613.1, C1614.1, C1615.2, C1617.2, C1618.2, U1601.17 (PGND1)
- net PG1: now also R3.1
- net V_{out1}: no longer U1601.26 (VOUT1)
- net V_{out2}: no longer C1615.1, R1608.1, U1601.5 (VOUT2)
- net Power channel 1/HB: now reaches U1601.20 (HB1)
- net at D1602.1 (K), U1601.11 (HB2): no longer C1612.1
- net at C1611.2: no longer U1601.36 (VDDA)
- net Power channel 1/SW: now reaches U1601.21 (SW1)
- net Power channel 1/LO: now reaches U1601.18 (LO1)
- net Power channel 1/LO: no longer U1601.19 (LOL1)
- net at C1613.2: no longer R1605.1
- net at L1602.2, Q1603.3 (S), Q1604.1 (D)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: no longer C1612.2
- net Power channel 1/HOL: now reaches U1601.23 (HOL1)
- net Power channel 1/HO: now reaches U1601.22 (HO1)
- net at C1609.1: no longer U1601.1 (SS2)
- net at C1608.1: no longer U1601.30 (SS1)
- net at C1610.1: no longer U1601.32 (RES)
- net Power channel 1/CS: now reaches U1601.27 (CS1)
- net at R1605.2, U1601.2 (COMP2): no longer C1614.2
- net Power channel 1/COMP: now reaches U1601.29 (COMP1)
- net FB1 renamed Power channel 1/FB
- new net: R1608.1, U1601.5 (VOUT2)
- new net Power channel 1/LOL: U1601.19 (LOL1)
- new net Power channel 1/PGND: U1601.17 (PGND1)
- new net Power channel 1/VOUT_FB: U1601.26 (VOUT1)
Other:
- added sheet Power channel 1 (power_channel.kicad_sch)
- company: (none) -> David Haisman
- title: (none) -> ${PROJECTNAME}
